Commit message: Updates

File: controller_ws/src/igvc_self_drive_sim/igvc_self_drive_description/urdf/gem.urdf.xacro (robot description, xacro)
@@ -14,5 +14,5 @@
   <xacro:property name="body_length" value="0.6" />
   <xacro:macro name="rear_wheel" params="name x y z flip" >
-    <link name="wheel_${name}" >
+    <link name="link_wheel_${name}" >
       <visual>
         <origin xyz="0 0 0" rpy="0 ${flip * pi - pi/2} 0" />
@@ -34,5 +34,5 @@
     <joint name="wheel_${name}" type="continuous" >
       <parent link="base_link" />
-      <child link="wheel_${name}" />
+      <child link="link_wheel_${name}" />
       <origin xyz="${x} ${y} ${z}" rpy="-1.57079632679 0 0" />
       <axis xyz="0 0 1" />
@@ -41,5 +41,5 @@
   </xacro:macro>
   <xacro:macro name="front_wheel" params="name x y z flip" >
-    <link name="wheel_${name}" >
+    <link name="link_wheel_${name}" >
       <visual>
         <origin xyz="0 0 0" rpy="0 ${flip * pi - pi/2} 0" />
@@ -56,8 +56,11 @@
         <origin xyz="0 0 0" rpy="0 0 0"/>
         <mass value="${wheel_mass}"/>
-        <inertia ixx="${wheel_mass/12*(3*wheel_radius*wheel_radius + wheel_thickness*wheel_thickness)}" ixy="0" ixz="0" iyy="${wheel_mass/12*(3*wheel_radius*wheel_radius + wheel_thickness*wheel_thickness)}" iyz="0" izz="${wheel_mass/2 * wheel_radius*wheel_radius}"/>
+        <inertia ixx="${wheel_mass/12*(3*wheel_radius*wheel_radius + wheel_thickness*wheel_thickness)}"
+          ixy="0" ixz="0"
+          iyy="${wheel_mass/12*(3*wheel_radius*wheel_radius + wheel_thickness*wheel_thickness)}"
+          iyz="0" izz="${wheel_mass/2 * wheel_radius*wheel_radius}"/>
       </inertial>
     </link>
-    <link name="steer_${name}" >
+    <link name="link_steer_${name}" >
       <inertial>
         <origin xyz="0 0 0" rpy="0 0 0"/>
@@ -68,5 +71,5 @@
     <joint name="steer_${name}" type="revolute" >
       <parent link="base_link" />
-      <child link="steer_${name}" />
+      <child link="link_steer_${name}" />
       <origin xyz="${x} ${y} ${z}" rpy="0 0 0" />
       <axis xyz="0 0 1" />
@@ -74,6 +77,6 @@
     </joint>
     <joint name="wheel_${name}" type="continuous" >
-      <parent link="steer_${name}" />
-      <child link="wheel_${name}" />
+      <parent link="link_steer_${name}" />
+      <child link="link_wheel_${name}" />
       <origin xyz="0 0 0" rpy="-1.57079632679 0 0" />
       <axis xyz="0 0 1" />

File: controller_ws/src/igvc_self_drive_sim/igvc_self_drive_description/urdf/gem_gazebo.urdf.xacro (robot description, xacro)
@@ -22,17 +22,17 @@
     <mu2>0.5</mu2>
   </gazebo>
-  <gazebo reference="wheel_fl" >
+  <gazebo reference="link_wheel_fl" >
     <mu1>${wheel_friction}</mu1>
     <mu2>${wheel_friction}</mu2>
   </gazebo>
-  <gazebo reference="wheel_fr" >
+  <gazebo reference="link_wheel_fr" >
     <mu1>${wheel_friction}</mu1>
     <mu2>${wheel_friction}</mu2>
   </gazebo>
-  <gazebo reference="wheel_rl" >
+  <gazebo reference="link_wheel_rl" >
     <mu1>${wheel_friction}</mu1>
     <mu2>${wheel_friction}</mu2>
   </gazebo>
-  <gazebo reference="wheel_rr" >
+  <gazebo reference="link_wheel_rr" >
     <mu1>${wheel_friction}</mu1>
     <mu2>${wheel_friction}</mu2>

File: controller_ws/src/igvc_self_drive_sim/igvc_self_drive_description/urdf/gem_sensors.urdf.xacro (robot description, xacro)
@@ -5,11 +5,31 @@
   <xacro:include filename="$(find igvc_self_drive_description)/urdf/sensors/camera.urdf.xacro" />
   <xacro:camera_sim name="camera_front" parent="base_footprint" >
-    <origin xyz="1.75 0 2.1" rpy="0 0.55 0" />
+    <origin xyz="1.75 0 2.1" rpy="0 0 0" />
+  </xacro:camera_sim>
+    <!-- Camera Back-->
+  <xacro:include filename="$(find igvc_self_drive_description)/urdf/sensors/camera_back.urdf.xacro" />
+  <xacro:camera_sim name="camera_back" parent="base_footprint" >
+    <origin xyz="0.25 0 2.1" rpy="0 0 3.1415926" />
+  </xacro:camera_sim>
+    <!-- Camera Left-->
+  <xacro:include filename="$(find igvc_self_drive_description)/urdf/sensors/camera_left.urdf.xacro" />
+  <xacro:camera_sim name="camera_left" parent="base_footprint" >
+    <origin xyz="1.65 0.56 2.1" rpy="0.0 0 0.6" />
+  </xacro:camera_sim>
+    <!-- Camera Right-->
+  <xacro:include filename="$(find igvc_self_drive_description)/urdf/sensors/camera_right.urdf.xacro" />
+  <xacro:camera_sim name="camera_right" parent="base_footprint" >
+    <origin xyz="1.65 -0.56 2.1" rpy="0. 0 -0.6" />
   </xacro:camera_sim>
   <!-- LIDAR -->
-  <xacro:include filename="$(find hector_sensors_description)/urdf/hokuyo_utm30lx.urdf.xacro" />
+<!--   <xacro:include filename="$(find hector_sensors_description)/urdf/hokuyo_utm30lx.urdf.xacro" />
   <xacro:hokuyo_utm30lx name="laser" parent="base_footprint" ros_topic="scan" update_rate="40" ray_count="720" min_angle="-90" max_angle="90" >
     <origin xyz="2.75 0 0.85" rpy="0 0 0" />
-  </xacro:hokuyo_utm30lx>
+  </xacro:hokuyo_utm30lx> -->
+  <!-- IMU -->
+  <xacro:include filename="$(find igvc_self_drive_description)/urdf/sensors/imu.urdf.xacro" />
+  <xacro:imu name="imu" parent="base_footprint" >
+    <origin xyz="1.20 0 1.2" rpy="0 0 0" />
+  </xacro:imu>
   <!-- GPS -->
   <xacro:include filename="$(find igvc_self_drive_description)/urdf/sensors/gps.urdf.xacro" />
@@ -17,5 +37,10 @@
     <origin xyz="0.8 0 2.35" rpy="0 0 0" />
   </xacro:gps>
-  <!-- Sonar sensors -->
+  <!--3D LIDAR-->
+  <xacro:include filename="$(find igvc_self_drive_description)/urdf/sensors/OS1-64.urdf.xacro"/>
+  <xacro:OS1-64 parent="base_footprint" hz="10" samples="220">
+    <origin xyz="1.30 0 2.50" rpy="0 0 0" />
+  </xacro:OS1-64>
+  <!-- Sonar sensors
   <xacro:include filename="$(find hector_sensors_description)/urdf/sonar_sensor.urdf.xacro" />
   <xacro:sonar_sensor name="front_center" parent="base_footprint" ros_topic="sonar/front_center" update_rate="20" min_range="0.1" max_range="2" field_of_view="0.17" ray_count="3" >
@@ -48,4 +73,4 @@
   <xacro:sonar_sensor name="right_side_rear" parent="base_footprint" ros_topic="sonar/right_side_rear" update_rate="20" min_range="0.1" max_range="2" field_of_view="0.17" ray_count="3" >
     <origin xyz="0 -0.71 0.71" rpy="0 0 ${-M_PI/2}" />
-  </xacro:sonar_sensor>
+  </xacro:sonar_sensor> -->
 </robot>

File: controller_ws/src/igvc_self_drive_sim/igvc_self_drive_description/urdf/sensors/camera.urdf.xacro (robot description, xacro)
@@ -16,5 +16,5 @@
       <parent link="${name}_optical" />
       <child link="${name}" />
-      <origin xyz="0 0 0" rpy="-1.57079632679 0 -1.57079632679" />
+      <origin xyz="0 0 0" rpy="0 0 0" />
     </joint>
     <joint name="${name}_joint" type="fixed" >
@@ -28,13 +28,13 @@
         <update_rate>30.0</update_rate>
         <camera name="cam">
-          <horizontal_fov>1.04</horizontal_fov>
+          <horizontal_fov>1.87</horizontal_fov>
           <image>
-            <width>640</width>
-            <height>480</height>
+            <width>1280</width>
+            <height>720</height>
             <format>R8G8B8</format>
           </image>
           <clip>
-            <near>0.02</near>
-            <far>300</far>
+            <near>0.05</near>
+            <far>60</far>
           </clip>
           <noise>
@@ -44,5 +44,5 @@
                  channels, which at that point lie in the range [0,1]. -->
             <mean>0.0</mean>
-            <stddev>0.007</stddev>
+            <stddev>0.0</stddev>
           </noise>
         </camera>
